Commit message: Update depends
Signed-off-by: Adam Krawczyk <adam-krawczyk@outlook.com>

File: Assets/urdf/tiago_robot/tiago_description/robots/tiago.urdf.xacro (robot description, xacro)
@@ -14,7 +14,7 @@
 <robot  xmlns:xacro="http://ros.org/wiki/xacro"
         name="tiago" >
-    <xacro:arg name="arm" default="right-arm"/> <!-- right-arm, left-arm, no-arm -->
+    <xacro:arg name="arm" default="right-arm"/> <!-- right-arm, no-arm -->
     <xacro:arg name="wrist_model" default="wrist-2010"/>
-    <xacro:arg name="end_effector" default="pal-hey5"/> <!-- no-end-effector, pal-gripper, pal-hey5, schunk-wsg-->
+    <xacro:arg name="end_effector" default="pal-hey5"/> <!-- no-end-effector, pal-gripper, pal-hey5-->
     <xacro:arg name="ft_sensor" default="schunk-ft"/> <!-- no-ft-sensor, schunk-ft -->
     <xacro:arg name="laser_model" default="sick-571"/> <!-- no-laser, hokuyo, sick-551, sick-561, sick-571-->
@@ -28,5 +28,5 @@
     <xacro:arg name="use_sim" default="true"/>
     <xacro:property name="arm" value="$(arg arm)" />
-    <xacro:if value="${arm not in ['right-arm', 'left-arm', 'no-arm']}">
+    <xacro:if value="${arm not in ['right-arm', 'no-arm']}">
       <xacro:wrong_arm/>
     </xacro:if>
@@ -45,5 +45,5 @@
     </xacro:if>
   </xacro:if>
-  <xacro:if value="${end_effector not in ['no-end-effector', 'pal-gripper', 'pal-hey5', 'schunk-wsg', 'custom']}">
+  <xacro:if value="${end_effector not in ['no-end-effector', 'pal-gripper', 'pal-hey5', 'custom']}">
     <xacro:wrong_end_effector/>
   </xacro:if>

File: Assets/urdf/tiago_robot/tiago_description/urdf/end_effector/end_effector.urdf.xacro (robot description, xacro)
@@ -31,19 +31,4 @@
     </xacro:pal_gripper>
   </xacro:if>
-  <!-- Schunk WSG -->
-  <!-- <xacro:if value="${type == 'schunk-wsg'}">
-    <xacro:include filename="$(find pal_wsg_gripper_description)/urdf/gripper.urdf.xacro" />
-    <xacro:include filename="$(find pal_wsg_gripper_description)/urdf/fingertip_sensor.urdf.xacro" />
-    <xacro:pal_wsg_gripper parent="${parent}" name="${name}">
-      <origin xyz="0.01 0 0" rpy="${90*deg_to_rad} ${90*deg_to_rad} ${-90*deg_to_rad}"/>
-    </xacro:pal_wsg_gripper> -->
-    <!-- Fingertip sensors -->
-    <!-- <xacro:fingertip_sensor name="${name}_left" parent="${name}_left_finger">
-      <origin xyz="0.035 0 -0.1465" rpy="0 ${-90*deg_to_rad} 0"/>
-    </xacro:fingertip_sensor>
-    <xacro:fingertip_sensor name="${name}_right" parent="${name}_right_finger">
-      <origin xyz="-0.035 0 -0.1465" rpy="0 ${90*deg_to_rad} 0"/>
-    </xacro:fingertip_sensor>
-  </xacro:if> -->
   <!-- Hand -->
   <xacro:if value="${type == 'pal-hey5'}">
